File: Schema/pH/PH_074_isolated_SMD_rev1_2.brd (EAGLE design)
At the start: 67 x 48 mm, 32 parts, among them IC1 TL074D, IC2 TLC271D

Commit message: add Shield
Parts:
- R6: value 2k2 -> 200R
- moved R8 22.9 mm to (40.4, 12.3), turned to 270 degrees
- moved LED1 16.5 mm to (46.0, 24.0)
- moved R5 10.6 mm to (41.5, 21.8), turned to 0 degrees
- moved D1 10.5 mm to (43.1, 12.3), turned to 90 degrees
- moved IL300 10.4 mm to (45.7, 36.7)
- moved R6 7.16 mm to (43.1, 17.7)
- moved PWS1 0.51 mm to (64.6, 17.6)
Connections:
- net -12V: no longer R6.1
- net GND: now also D1.1
- net N$8: now also R6.1; no longer D1.1
Routing:
- net N$7: track 41.8 -> 5.06 mm
- net N$9: track 8.43 -> 21.8 mm
- net N$4: track 19.5 -> 30.7 mm
- net N$21: track 22.4 -> 11.7 mm
- net N$8: track 13.7 -> 5.59 mm
- net -12V: track 45.7 -> 53.1 mm
- net +12V: track 80.8 -> 87.2 mm
Other:
- board text added: "pH rev 1.2"
- board text removed: "pH rev 1.1"

Commit message: schema upload
Parts:
- moved IL300 0.40 mm to (45.7, 37.1)
Routing:
- net N$4: track 30.7 -> 32.2 mm
- net +12V: track 87.2 -> 88.5 mm
- net N$21: track 11.7 -> 11.0 mm
